File: hardware/pi_dsm_26_2.kicad_sch (KiCad schematic)
At the start: 17 parts, among them J1 Tomada fêmea NBR 14136, J3 Borne de aterramento DIN verd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, K3 Módulo relé 5 V, 2 canais (1 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, P1 Cabo macho NBR 14136, SW1 Botão momentâneo, U1 ESP32 DevKit V1 (30 pinos), U2 HLK-PM01

Commit message: fix(hardware): corrigir símbolo ESP32_30pin, pull-up R1 e remover PWR_FLAG (#20, #131)
- ESP32_30Pin: pino 16 (3.3v) corrigido para power_out (em esp32_30pin.kicad_sym e no .kicad_sch)
- Removido o PWR_FLAG (#FLG02) e o +3V3 redundante que compensavam a falta de power_out no pino 16
- R1: reorientado o símbolo +3V3 (#PWR08) na vertical com rotação 0 (apontando para cima no topo de R1), eliminando a rotação invertida 180°
- RELE_IN: roteada a linha de sinal para a perna inferior de R1 e posicionado o label de forma limpa abaixo de K3
- Regenerado hardware/pi_dsm_26_2.pdf com kicad-cli 10.0.5; ERC validado com 0 erros e 22 avisos esperados

Closes #20
Closes #131
Connections:
- net +3V3: now also R1.1; no longer R1.2
- net RELE_IN: now also R1.2; no longer R1.1
Changed lines of the file:
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@@
 	)
 	(junction
-		(at 128.27 66.04)
-		(diameter 0)
-		(color 0 0 0 0)
-	)
-	(junction
 		(at 83.82 132.08)
 		(diameter 0)
@@
 	(wire
 		(pts
-			(xy 134.62 66.04) (xy 134.62 71.12)
+			(xy 134.62 67.31) (xy 134.62 71.12)
 		)
 		(stroke
@@
 	(wire
 		(pts
-			(xy 45.72 33.02) (xy 45.72 38.1)
-		)
-		(stroke
-			(width 0)
-			(type default)
-		)
-	)
-	(wire
-		(pts
 			(xy 128.27 60.96) (xy 140.97 60.96)
 		)
@@
 	(wire
 		(pts
-			(xy 128.27 66.04) (xy 134.62 66.04)
+			(xy 128.27 66.04) (xy 128.27 82.55)
 		)
 		(stroke
@@
 	(wire
 		(pts
-			(xy 231.14 143.51) (xy 236.22 143.51)
+			(xy 128.27 82.55) (xy 134.62 82.55)
 		)
 		(stroke
@@
 	(wire
 		(pts
-			(xy 83.82 132.08) (xy 87.63 132.08)
+			(xy 231.14 143.51) (xy 236.22 143.51)
 		)
 		(stroke
@@
 	(wire
 		(pts
-			(xy 127 66.04) (xy 128.27 66.04)
+			(xy 83.82 132.08) (xy 87.63 132.08)
 		)
 		(stroke
@@
 	)
 	(label "RELE_IN"
-		(at 127 66.04 0)
+		(at 128.27 73.66 180)
 		(effects
 			(font
 				(size 1.27 1.27)
 			)
-			(justify left bottom)
+			(justify right bottom)
 		)
 	)
@@
 	(symbol
 		(lib_id "power:+3V3")
-		(at 134.62 82.55 180)
+		(at 134.62 67.31 0)
 		(unit 1)
 		(body_style 1)
@@
 		(dnp no)
 		(property "Reference" "#PWR08"
-			(at 134.62 82.55 0)
+			(at 134.62 67.31 0)
 			(hide yes)
 			(show_name no)
@@
 		)
 		(property "Value" "+3V3"
-			(at 134.62 86.36 0)
+			(at 134.62 63.5 0)
 			(show_name no)
 			(do_not_autoplace no)
@@
 		)
 		(property "Footprint" ""
-			(at 134.62 82.55 0)
+			(at 134.62 67.31 0)
 			(hide yes)
 			(show_name no)
@@
 		)
 		(property "Datasheet" ""
-			(at 134.62 82.55 0)
+			(at 134.62 67.31 0)
 			(hide yes)
 			(show_name no)
@@
 		)
 		(property "Description" ""
-			(at 134.62 82.55 0)
+			(at 134.62 67.31 0)
 			(show_name no)
 			(do_not_autoplace no)
@@
 	)
 	(symbol
-		(lib_id "power:PWR_FLAG")
-		(at 45.72 38.1 180)
-		(unit 1)
-		(body_style 1)
-		(exclude_from_sim no)
-		(in_bom yes)
-		(on_board yes)
-		(in_pos_files yes)
-		(dnp no)
-		(property "Reference" "#FLG02"
-			(at 45.72 38.1 0)
-			(hide yes)
-			(show_name no)
-			(do_not_autoplace no)
-			(effects
-				(font
-					(size 1.27 1.27)
-				)
-			)
-		)
-		(property "Value" "PWR_FLAG"
-			(at 45.72 38.1 0)
-			(hide yes)
-			(show_name no)
-			(do_not_autoplace no)
-			(effects
-				(font
-					(size 1.27 1.27)
-				)
-			)
-		)
-		(property "Footprint" ""
-			(at 45.72 38.1 0)
-			(hide yes)
-			(show_name no)
-			(do_not_autoplace no)
-			(effects
-				(font
-					(size 1.27 1.27)
-				)
-			)
-		)
-		(property "Datasheet" ""
-			(at 45.72 38.1 0)
-			(hide yes)
-			(show_name no)
-			(do_not_autoplace no)
-			(effects
-				(font
-					(size 1.27 1.27)
-				)
-			)
-		)
-		(property "Description" ""
-			(at 45.72 38.1 0)
-			(show_name no)
-			(do_not_autoplace no)
-			(effects
-				(font
-					(size 1.27 1.27)
-				)
-			)
-		)
-		(pin "1"
-		)
-		(instances
-			(project "pi_dsm_26_2"
-				(path "/b44094fb-e67c-4704-b1f1-1092cb00b967"
-					(reference "#FLG02")
-					(unit 1)
-				)
-			)
-		)
-	)
-	(symbol
 		(lib_id "Connector_Generic:Conn_01x01")
 		(at 228.6 26.67 0)
@@
 					(unit 1)
 				)
-			)
-		)
-	)
-	(symbol
-		(lib_id "power:+3V3")
-		(at 45.72 33.02 0)
-		(unit 1)
-		(body_style 1)
-		(exclude_from_sim no)
-		(in_bom yes)
-		(on_board yes)
-		(in_pos_files yes)
-		(dnp no)
-		(property "Reference" "#PWR18"
-			(at 45.72 33.02 0)
-			(hide yes)
-			(show_name no)
-			(do_not_autoplace no)
-			(effects
-				(font
-					(size 1.27 1.27)
-				)
-			)
-		)
-		(property "Value" "+3V3"
-			(at 45.212 28.448 0)
-			(show_name no)
-			(do_not_autoplace no)
-			(effects
-				(font
-					(size 1.27 1.27)
-				)
-			)
-		)
-		(property "Footprint" ""
-			(at 45.72 33.02 0)
-			(hide yes)
-			(show_name no)
-			(do_not_autoplace no)
-			(effects
-				(font
-					(size 1.27 1.27)
-				)
-			)
-		)
-		(property "Datasheet" ""
-			(at 45.72 33.02 0)
-			(hide yes)
-			(show_name no)
-			(do_not_autoplace no)
-			(effects
-				(font
-					(size 1.27 1.27)
-				)
-			)
-		)
-		(property "Description" ""
-			(at 45.72 33.02 0)
-			(show_name no)
-			(do_not_autoplace no)
-			(effects
-				(font
-					(size 1.27 1.27)
-				)
-			)
-		)
-		(pin "1"
-		)
-		(instances
-			(project "pi_dsm_26_2"
-				(path "/b44094fb-e67c-4704-b1f1-1092cb00b967"
-					(reference "#PWR18")
-					(unit 1)
-				)
